File: ESP32Clone/ESP32Clone.kicad_pcb (KiCad board)
At the start: 2 copper layers, 53.3 x 29.2 mm, 58 parts, among them J1 Connector, USB-TYPE-C-16P, J2 Conn_01x08_Pin, J3 Conn_01x08_Pin, U1 TPS54331DR, U2 ESP32-C3FH4, U3 AHT20, U4 BH1750FVI-TR, U5 24LC1025-I_SM, X1 40MHz, 15pF

Commit message: removed a few islands and generated bom
Routing:
- net GND: vias 142 -> 150
Other:
- board text added: "Made on 1-16-2026"
- board text removed: "Made on <date>"
Changed lines of the file:
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@@
 		)
 	)
-	(gr_text "Made on <date>"
+	(gr_text "Made on 1-16-2026"
 		(at 100.8888 42.8244 0)
 		(layer "B.SilkS")
@@
 	)
 	(via
+		(at 121.158 37.1348)
+		(size 0.6)
+		(drill 0.3)
+		(layers "F.Cu" "B.Cu")
+		(free yes)
+		(net 1)
+	)
+	(via
 		(at 125.222 35.56)
 		(size 0.6)
@@
 	)
 	(via
+		(at 96.6724 41.8084)
+		(size 0.6)
+		(drill 0.3)
+		(layers "F.Cu" "B.Cu")
+		(free yes)
+		(net 1)
+	)
+	(via
 		(at 94.488 19.558)
 		(size 0.6)
@@
 	)
 	(via
+		(at 96.2152 42.418)
+		(size 0.6)
+		(drill 0.3)
+		(layers "F.Cu" "B.Cu")
+		(free yes)
+		(net 1)
+	)
+	(via
 		(at 87.63 26.035)
 		(size 0.6)
@@
 	)
 	(via
+		(at 116.078 37.7444)
+		(size 0.6)
+		(drill 0.3)
+		(layers "F.Cu" "B.Cu")
+		(free yes)
+		(net 1)
+	)
+	(via
 		(at 117.475 25.4)
 		(size 0.6)
@@
 	)
 	(via
+		(at 95.4532 23.5204)
+		(size 0.6)
+		(drill 0.3)
+		(layers "F.Cu" "B.Cu")
+		(free yes)
+		(net 1)
+	)
+	(via
 		(at 101.346 42.926)
 		(size 0.6)
@@
 	)
 	(via
+		(at 99.7204 42.5704)
+		(size 0.6)
+		(drill 0.3)
+		(layers "F.Cu" "B.Cu")
+		(free yes)
+		(net 1)
+	)
+	(via
 		(at 114.935 25.4)
 		(size 0.6)
@@
 	)
 	(via
+		(at 104.5972 30.3276)
+		(size 0.6)
+		(drill 0.3)
+		(layers "F.Cu" "B.Cu")
+		(free yes)
+		(net 1)
+	)
+	(via
 		(at 116.84 27.305)
 		(size 0.6)
@@
 	)
 	(via
+		(at 95.758 42.1132)
+		(size 0.6)
+		(drill 0.3)
+		(layers "F.Cu" "B.Cu")
+		(free yes)
+		(net 1)
+	)
+	(via
 		(at 91.44 32.004)
 		(size 0.6)
@@
 	)
 	(via
-		(at 105.5312 34.757228)
+		(at 105.5312 34.757227)
 		(size 0.6)
 		(drill 0.3)
@@
 	)
 	(segment
-		(start 105.5312 34.757228)
-		(end 105.5312 34.76)
+		(start 108.688 36.6)
+		(end 109.483535 36.6)
 		(width 0.2)
 		(layer "B.Cu")
@@
 	)
 	(segment
-		(start 105.5312 34.76)
-		(end 105.7436 34.9724)
+		(start 108.664 36.576)
+		(end 108.688 36.6)
 		(width 0.2)
 		(layer "B.Cu")
@@
 	)
 	(segment
-		(start 105.7436 34.9724)
-		(end 105.7436 35.1316)
+		(start 105.5312 34.757227)
+		(end 105.5312 34.76)
 		(width 0.2)
 		(layer "B.Cu")
@@
 	)
 	(segment
-		(start 109.483535 36.6)
-		(end 109.541768 36.541768)
+		(start 105.7436 34.9724)
+		(end 105.7436 35.1316)
 		(width 0.2)
 		(layer "B.Cu")
@@
 	)
 	(segment
-		(start 123.643434 38.356566)
-		(end 123.941964 38.058036)
+		(start 105.7436 35.1316)
+		(end 107.188 36.576)
 		(width 0.2)
 		(layer "B.Cu")
@@
 	)
 	(segment
-		(start 108.688 36.6)
-		(end 109.483535 36.6)
+		(start 105.5312 34.76)
+		(end 105.7436 34.9724)
 		(width 0.2)
 		(layer "B.Cu")
@@
 	)
 	(segment
-		(start 105.7436 35.1316)
-		(end 107.188 36.576)
+		(start 109.483535 36.6)
+		(end 109.541768 36.541768)
 		(width 0.2)
 		(layer "B.Cu")
@@
 	)
 	(segment
-		(start 108.664 36.576)
-		(end 108.688 36.6)
+		(start 123.643434 38.356566)
+		(end 123.941964 38.058036)
 		(width 0.2)
 		(layer "B.Cu")
